File: pcb/schmitt_ladder.sch (KiCad schematic (older format))
At the start: 56 parts, among them J1 CV_00 IN, J2 CV_01 IN, J3 GATE_IN, J4 Eurorack Power, J5 TFT DISPLAY, J6 STEMMA-QT, J7 CV_00 OUT, J8 CV_01 OUT, M1 ItsyBitsy_M4_Express, U1 OPA2156xDGK, U2 OPA2156xDGK, U3 LM1117-5.0, U4 OPA2156xDGK, U5 OPA2156xDGK

Commit message: test new algorithm; update ladder schematic
Parts:
- removed BZ1: PS1240P02BT, digikey-footprints:Piezo_Transducer_THT_PS1240P02BT, symbol dk_Alarms-Buzzers-and-Sirens:PS1240P02BT
- removed C1, C3, C5: 0.1uF, Capacitor_SMD:C_0805_2012Metric, symbol Range_Slicer_PCB-rescue:C_Small-device-2019-04-06_Range_Slicer_PCB-rescue
- removed C2, C4, C6: 10uF, Capacitor_SMD:C_1210_3225Metric, symbol Range_Slicer_PCB-rescue:CP1_Small-device-2019-04-06_Range_Slicer_PCB-rescue
- removed C7, C8: 18pF, Capacitor_SMD:C_0805_2012Metric, symbol Range_Slicer_PCB-rescue:C_Small-device-2019-04-06_Range_Slicer_PCB-rescue
- removed D10: CV_01_IN_RED, LED_THT:LED_D3.0mm, symbol Range_Slicer_PCB-rescue:LED-device-2019-04-06_Range_Slicer_PCB-rescue
- removed D11: GATE_RED, LED_THT:LED_D3.0mm, symbol Range_Slicer_PCB-rescue:LED-device-2019-04-06_Range_Slicer_PCB-rescue
- removed D12, D7, D8: B160, Diode_SMD:D_SMA, symbol Range_Slicer_PCB-rescue:B160-E3-diode-2019-04-06_Range_Slicer_PCB-rescue
- removed D14: SEL_ENC_GRN, LED_THT:LED_D3.0mm, symbol Range_Slicer_PCB-rescue:LED-device-2019-04-06_Range_Slicer_PCB-rescue
- removed D15: PWR, LED_THT:LED_D3.0mm, symbol Range_Slicer_PCB-rescue:LED-device-2019-04-06_Range_Slicer_PCB-rescue
- removed D16, D17: CV_00_OUT_RED, LED_THT:LED_D3.0mm, symbol Range_Slicer_PCB-rescue:LED-device-2019-04-06_Range_Slicer_PCB-rescue
- removed D9: CV_00_IN_RED, LED_THT:LED_D3.0mm, symbol Range_Slicer_PCB-rescue:LED-device-2019-04-06_Range_Slicer_PCB-rescue
- removed DA1, DA2: BAT54XY, Package_TO_SOT_SMD:SOT-363_SC-70-6, symbol Adafruit_custom:BAT54XY_Dual_Schottky_Diode_Array
- removed J1: CV_00 IN, Adafruit:Schurter_4832.2211_3.5mm_vert_TS_switch, symbol Adafruit_custom:Schurter_4832.2211_3.5mm_vert_TS_switch
- removed J2: CV_01 IN, Adafruit:Schurter_4832.2211_3.5mm_vert_TS_switch, symbol Adafruit_custom:Schurter_4832.2211_3.5mm_vert_TS_switch
- removed J3: GATE_IN, Adafruit:Schurter_4832.2211_3.5mm_vert_TS_switch, symbol Adafruit_custom:Schurter_4832.2211_3.5mm_vert_TS_switch
- removed J4: Eurorack Power, Connector_IDC:IDC-Header_2x05_P2.54mm_Vertical, symbol Connector_Generic:Conn_02x05_Odd_Even
- removed J5: TFT DISPLAY, Adafruit:TFT_Display_1.44in_128x128_PID2088, symbol Connector_Generic:Conn_01x11
- removed J6: STEMMA-QT, Connector_JST:JST_SH_SM04B-SRSS-TB_1x04-1MP_P1.00mm_Horizontal, symbol Range_Slicer_PCB-rescue:CONN_01X04-conn-2019-04-06_Range_Slicer_PCB-rescue
- removed J7: CV_00 OUT, Adafruit:Schurter_4832.2211_3.5mm_vert_TS_switch, symbol Adafruit_custom:Schurter_4832.2211_3.5mm_vert_TS_switch
- removed J8: CV_01 OUT, Adafruit:Schurter_4832.2211_3.5mm_vert_TS_switch, symbol Adafruit_custom:Schurter_4832.2211_3.5mm_vert_TS_switch
- removed M1: ItsyBitsy_M4_Express, Adafruit:ItsyBitsy M4 Express, symbol Adafruit_custom:ItsyBitsy_M4_Express
- removed R1: 470, Resistor_SMD:R_0805_2012Metric, symbol Range_Slicer_PCB-rescue:R_Small-device-2019-04-06_Range_Slicer_PCB-rescue
- removed R10, R12, R8, R9: 665, Resistor_SMD:R_0805_2012Metric, symbol Range_Slicer_PCB-rescue:R_Small-device-2019-04-06_Range_Slicer_PCB-rescue
- removed R11: 1K, Resistor_SMD:R_0805_2012Metric, symbol Range_Slicer_PCB-rescue:R_Small-device-2019-04-06_Range_Slicer_PCB-rescue
- removed R13: 1.5K, Resistor_SMD:R_0805_2012Metric, symbol Range_Slicer_PCB-rescue:R_Small-device-2019-04-06_Range_Slicer_PCB-rescue
- removed R14: 20K, Resistor_SMD:R_0805_2012Metric, symbol Range_Slicer_PCB-rescue:R_Small-device-2019-04-06_Range_Slicer_PCB-rescue
- removed R16, R17: 2K, Resistor_SMD:R_0805_2012Metric, symbol Range_Slicer_PCB-rescue:R_Small-device-2019-04-06_Range_Slicer_PCB-rescue
- removed R2, R3, R7: 10K, Resistor_SMD:R_0805_2012Metric, symbol Range_Slicer_PCB-rescue:R_Small-device-2019-04-06_Range_Slicer_PCB-rescue
- removed R4, R5, R6: 5.05K, Resistor_SMD:R_0805_2012Metric, symbol Range_Slicer_PCB-rescue:R_Small-device-2019-04-06_Range_Slicer_PCB-rescue
- removed ROT1: SELECT, digikey-footprints:Rotary_Encoder_Switched_PEC11R_mntg_hole, symbol Range_Slicer_PCB-rescue:PEC11R-4215F-S0024-dk_Encoders-2019-04-06_Range_Slicer_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
- removed RV1, RV2: 100K, Adafruit:Potentiometer_Trimmer_Bourns_PV36W, symbol Range_Slicer_PCB-rescue:POT-device-2019-04-06_Range_Slicer_PCB-rescue
- removed U1, U5: OPA2156xDGK, Package_SO:VSSOP-8_3.0x3.0mm_P0.65mm, symbol Amplifier_Operational:OPA2156xDGK
- removed unit 3 of U2
- removed U3: LM1117-5.0, Package_TO_SOT_SMD:SOT-223-3_TabPin2, symbol Range_Slicer_PCB-rescue:LM1117-5.0-regul-2019-04-06_Range_Slicer_PCB-rescue
- removed unit 3 of U4
- added R1, R11, R14, R2, R5, R8: 10K, Resistor_SMD:R_0805_2012Metric, symbol schmitt_ladder-rescue:R_Small-device-2019-04-06_Range_Slicer_PCB-rescue-Range_S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
- added R10, R12, R13, R15, R16, R17, R18, R6, R7, R9: 100K, Resistor_SMD:R_0805_2012Metric, symbol schmitt_ladder-rescue:R_Small-device-2019-04-06_Range_Slicer_PCB-rescue-Range_S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
- added U3: OPA2156xDGK, Package_SO:VSSOP-8_3.0x3.0mm_P0.65mm, symbol Amplifier_Operational:OPA2156xDGK
- R3: renamed from R15; value 20K -> 100K; symbol Range_Slicer_PCB-rescue:R_Small-device-2019-04-06_Range_Slicer_PCB-rescue -> schmitt_ladder-rescue:R_Small-device-2019-04-06_Range_Slicer_PCB-rescue-Range_Slicer_PCB-rescue
- R4: renamed from R18; value 1K -> 100K; symbol Range_Slicer_PCB-rescue:R_Small-device-2019-04-06_Range_Slicer_PCB-rescue -> schmitt_ladder-rescue:R_Small-device-2019-04-06_Range_Slicer_PCB-rescue-Range_Slicer_PCB-rescue
- renumbered U4 to U1
Connections:
- net CV_00_OUT is gone; now on net INPUT: U1.3 (+)
- net GATE_IN is gone; now on net INPUT: U2.3 (+)
- net SEL_ENC is gone; now on net INPUT: U2.5 (+)
- net GND: now also R12.2, R14.1, R15.2, R17.2, R6.2, R9.2, U3.6 (-)
- net at U1.2 (-): now also R1.1, R2.2
- net at U1.6 (-): now also R2.1, R5.2
- net SLICE_n-1: now reaches U1.7
- net SLICE_n-1: now also R7.1
- net INPUT: now reaches U1.5 (+)
- net INPUT: now also R3.1, R4.2, R10.2, R12.1, R13.2, R15.1, R16.2, R17.1, R18.2, R6.1, R7.2, R9.1, U3.3 (+), U3.5 (+); no longer U1.1
- net at U2.6 (-): now also R11.2, R8.1
- net SLICE_n-3: now reaches U2.7
- net SLICE_n-3: now also R13.1
- net SLICE_n-2: now reaches U2.1
- net SLICE_n-2: now also R10.1
- net at U2.2 (-): now also R5.1, R8.2
- net SLICE_n: now reaches R4.1
- net SLICE_n: now also U1.1
- new net: R11.1, R14.2, U3.2 (-)
- new net +10V: R1.2
- new net SLICE_0: R18.1, U3.7
- new net SLICE_n-4: R16.1, U3.1
- no-connect marks 14 -> 0
Other:
- note removed: "3Vo"
- note removed: "Adafruit #2088\nColor 1.44-inch\n128x128 TFT display"
- note removed: "CV_00 Input"
- note removed: "CV_00 Output"
- note removed: "CV_01 Input"
- note removed: "CV_01 Output"
- note removed: "DC"
- note removed: "ENCODER Select"
- note removed: "Full-Scale\nCalibrate"
- note removed: "GATE Input"
- note removed: "Gnd"
- note removed: "Ideal gain = 3.03 = 10V Vout / 3.3V Vin\nset cal pot to ~~ 40.6K"
- note removed: "Input Signals"
- note removed: "Lite"
- note removed: "MISO"
- note removed: "MOSI"
- note removed: "Output Signals"
- note removed: "Panel\nPower\nIndicator"
- note removed: "Power Management"
- note removed: "Rotary Encoder"
- note removed: "Rst"
- note removed: "SCK"
- note removed: "SDCS"
- note removed: "STEMMA-QT Interface\nJST-SH"
- note removed: "TFTCS"
- note removed: "Vf = 3v"
- note removed: "Vin"
- moved on the sheet: R3, R4, U1A, U1B

Commit message: working on algorithm 4
Parts:
- removed R2: 10K, Resistor_SMD:R_0805_2012Metric, symbol schmitt_ladder-rescue:R_Small-device-2019-04-06_Range_Slicer_PCB-rescue-Range_S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
- removed R3, R4: 100K, Resistor_SMD:R_0805_2012Metric, symbol schmitt_ladder-rescue:R_Small-device-2019-04-06_Range_Slicer_PCB-rescue-Range_S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
- removed U2, U3: OPA2156xDGK, Package_SO:VSSOP-8_3.0x3.0mm_P0.65mm, symbol Amplifier_Operational:OPA2156xDGK
- added R14, R15, R16: 1K, Resistor_SMD:R_0805_2012Metric, symbol schmitt_ladder-rescue:R_Small-device-2019-04-06_Range_Slicer_PCB-rescue-Range_S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
- added R19, R20, R21: 100K, Resistor_SMD:R_0805_2012Metric, symbol schmitt_ladder-rescue:R_Small-device-2019-04-06_Range_Slicer_PCB-rescue-Range_S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
- added unit 3 of U1
- added U2: LM339, symbol Comparator:LM339
- added U3: LM4125IM5-2.0, Package_TO_SOT_SMD:SOT-23-5, symbol Reference_Voltage:LM4125IM5-2.0
- R1: value 10K -> 1K
- R17: value 100K -> 1K
- R2: renamed from R5; value 10K -> 1K
- R3: renamed from R8; value 10K -> 1K
- R4: renamed from R11; value 10K -> 1K
- R5: renamed from R14; value 10K -> 1K
- renumbered R7 to R10, R10 to R11, R13 to R12, R16 to R13, R9 to R7, R12 to R8, R15 to R9
Connections:
- net +10V: now also U1.8 (V+), U2.3 (V+), U3.4 (Vin)
- net GND: now also U1.4 (V-), U2.12 (V-), U3.2 (GND); no longer R17.2, R6.2, R7.2, R8.2, R9.2
- net INPUT: no longer R10.2, R11.2, R12.2, R13.2, R17.1, R18.2, R6.1, R7.1, R8.1, R9.1, U1.5 (+)
- net at R1.1: now also R2.2, U2.8 (-); no longer U1.2 (-)
- net OUTPUT: now reaches U1.6 (-)
- net OUTPUT: now also U1.7; no longer R2.2
- net at R2.1, R3.2: now also U2.10 (-)
- net at R3.1, R4.2: now also U2.6 (-)
- net at R4.1, R5.2: now also U2.4 (-)
- net SLICE_0 renamed SLICE_SUM
- net SLICE_SUM: now also U1.5 (+), R19.1, R20.1, R21.1
- net SLICE_n: no longer names the net of U1.1
- net SLICE_n: now also R6.2, R7.2, R8.2, R9.2, U1.2 (-)
- net SLICE_n-1 renamed SLICE_4
- net SLICE_4: now also R18.2, R14.1, U2.14; no longer U1.7
- net SLICE_n-2 renamed SLICE_3
- net SLICE_3: now also R15.1, R19.2, U2.13
- net SLICE_n-3 renamed SLICE_2
- net SLICE_2: now also R16.1, R20.2, U2.1
- net SLICE_n-4 renamed SLICE_1
- net SLICE_1: now also R17.1, R21.2, U2.2
- new net: R13.2, R9.1, U2.5 (+)
- new net: R12.2, R8.1, U2.7 (+)
- new net: R11.2, R7.1, U2.11 (+)
- new net: R10.2, R6.1, U2.9 (+)
- new net 2vREF: R14.2, R15.2, R16.2, R17.2, U3.5 (Vout)
Other:
- moved on the sheet: R1, R10, R11, R12, R13, R2, R3, R4, R5, R6, R7, R8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
